File: V 2.2/PCB/Spikeling_V2.2.kicad_pcb (KiCad board)
At the start: 2 copper layers, 120 x 80 mm, 51 parts

Commit message: general update
Parts:
- Current In: footprint Connector_Audio:Spikeling Audio Jack 3.5mm -> Audio_Module:Spikeling Audio Jack 3.5mm
- Stimulus Out: footprint Connector_Audio:Spikeling Audio Jack 3.5mm -> Audio_Module:Spikeling Audio Jack 3.5mm
- Synapse In 1: footprint Connector_Audio:Spikeling Audio Jack 3.5mm -> Audio_Module:Spikeling Audio Jack 3.5mm
- Synapse In 2: footprint Connector_Audio:Spikeling Audio Jack 3.5mm -> Audio_Module:Spikeling Audio Jack 3.5mm
- Synapse Out: footprint Connector_Audio:Spikeling Audio Jack 3.5mm -> Audio_Module:Spikeling Audio Jack 3.5mm
- moved Stimulus Out 0.39 mm to (214.0, 130.0)
- moved Synapse In 1 0.32 mm to (100.0, 56.1)
- moved Synapse In 2 0.25 mm to (100.0, 90.0)
- renumbered REF** to ESP32
Connections:
- Synapse In 1 pad : GNDREF -> (no net)
- Synapse In 2 pad : GNDREF -> (no net)
Routing:
- net VCC: track 392.8 -> 387.6 mm
- net /105: track 160.4 -> 155.4 mm
- net /104: track 144.3 -> 139.7 mm
- net /26: track 82.5 -> 86.8 mm
- net Net-(10Ω_RC1-Pad2): track 15.0 -> 18.4 mm
- net /200: track 43.9 -> 47.2 mm
- net /101: track 46.4 -> 43.3 mm
- net /203: track 38.3 -> 41.3 mm
- net /201: track 20.4 -> 23.4 mm
- net Net-(100Ω_Stim-LED1-Pad2): track 37.5 -> 39.7 mm
- net /35: track 87.9 -> 89.9 mm
- net /34: track 88.6 -> 90.4 mm
