File: V 2.2/PCB/Spikeling_V2.2.kicad_pcb (KiCad board)
At the start: 2 copper layers, 120 x 80 mm, 51 parts

Commit message: update pcb
Changed lines of the file:
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@@
   (footprint "Audio_Module:Spikeling_Photoreceptor" (layer "F.Cu")
     (at 159.6 122.9)
-    (fp_text reference "Photodiode Gain" (at 0 -0.5 unlocked) (layer "F.SilkS")
+    (fp_text reference "Photodiode Gain" (at 0.4 -8.6 unlocked) (layer "F.SilkS")
       (effects (font (size 1 1) (thickness 0.15)))
     )

Commit message: update pcb
Parts:
- .: renamed from Photodiode Gain
- BZ1: renamed from Spike Buzzer; value BZ1 -> Spike Buzzer
- C3: renamed from 1nF; value C3 -> 1nF RC
- D1: renamed from Photodiode; value D1 -> Photodiode
- D10: renamed from 9; value D10 -> Mode9
- D11: renamed from 10; value D11 -> Mode10
- D12: renamed from 11; value D12 -> Mode11
- D13: renamed from 12; value D13 -> Mode12
- D14: renamed from Spike_LED; value RGB -> Spike LED
- D2: renamed from 1; value D2 -> Mode1
- D3: renamed from 2; value D3 -> Mode2
- D4: renamed from 3; value D4 -> Mode3
- D5: renamed from 4; value D5 -> Mode4
- D6: renamed from 5; value D6 -> Mode5
- D7: renamed from 6; value D7 -> Mode6
- D8: renamed from 7; value D8 -> Mode7
- D9: renamed from 8; value LED -> Mode8
- J1: renamed from Synapse Out; value J1 -> Synapse Out
- J2: renamed from Synapse In 1; value J2 -> Synapse in 1
- J3: renamed from Synapse In 2; value J3 -> Synapse in 2
- J4: renamed from Current In; value J4 -> Current in
- J5: renamed from Stimulus Out; value J5 -> Stimulus Out
- R1: renamed from 10Ω; value R1 -> 10Ω RC
- R2: renamed from 10kΩ; value R2 -> 10kΩ PD pull-down
- R3: renamed from 100Ω; value R3 -> 100Ω Stim-LED
- R4: renamed from 100Ω; value R4 -> 100Ω Spike-LED
- R5: renamed from 10kΩ; value R5 -> 10kΩ SW pull-down
- R6: renamed from 100Ω; value R6 -> 100Ω_CharliePlex1
- R7: renamed from 100Ω; value R7 -> 100Ω_CharliePlex2
- R8: renamed from 100Ω; value R8 -> 100Ω_CharliePlex3
- R9: renamed from 100Ω; value R9 -> 100Ω_CharliePlex4
- RV1: renamed from Synapse1 Gain; value RV1 -> Synapse 1 Gain
- RV2: renamed from Synapse2 Gain; value RV2 -> Synapse 2 Gain
- RV3: renamed from Voltage Membrane; value RV3 -> Voltage Membrane
- RV4: renamed from Noise; value RV4 -> Noise
- RV5: renamed from Photodiode Gain; value RV5 -> Photodiode Gain
- RV6: renamed from Stimulus; value RV6 -> Stimulus Strength
- RV7: renamed from Stimulus; value RV7 -> Stimulus Frequency
- SW1: renamed from Mode Button; value SW1 -> Mode Button
- SW2: renamed from Reset Button; value SW2 -> Reset Button
- U1: renamed from ESP32 Wroom-32 Dev Module
- renumbered 1μF to C1, 1μF to C2, MCP3208 to U2, MCP3208 to U3
Other:
- board text removed: "Frequency"
- board text removed: "Strength"

Commit message: Update Spikeling_V2.2.kicad_pcb
Parts:
- C3: value 1nF RC -> 1nF
- R1: value 10Ω RC -> 10Ω
- R2: value 10kΩ PD pull-down -> 10kΩ
- R3: value 100Ω Stim-LED -> 100Ω
- R4: value 100Ω Spike-LED -> 100Ω
- R5: value 10kΩ SW pull-down -> 10kΩ
- R6: value 100Ω_CharliePlex1 -> 100Ω
- R7: value 100Ω_CharliePlex2 -> 100Ω
- R8: value 100Ω_CharliePlex3 -> 100Ω
- R9: value 100Ω_CharliePlex4 -> 100Ω
Changed lines of the file:
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@@
       (effects (font (size 0.75 0.75) (thickness 0.1)))
     )
-    (fp_text value "10kΩ SW pull-down" (at 5.08 0.1 180) (layer "F.SilkS")
+    (fp_text value "10kΩ" (at 5.08 0.1 180) (layer "F.SilkS")
       (effects (font (size 1 1) (thickness 0.15)))
     )
@@
       (effects (font (size 0.75 0.75) (thickness 0.1)))
     )
-    (fp_text value "100Ω Stim-LED" (at 5.1 0.1) (layer "F.SilkS")
+    (fp_text value "100Ω" (at 5.1 0.1) (layer "F.SilkS")
       (effects (font (size 1 1) (thickness 0.15)))
     )
@@
       (effects (font (size 0.75 0.75) (thickness 0.1)))
     )
-    (fp_text value "100Ω_CharliePlex4" (at 5.1 0.1) (layer "F.SilkS")
+    (fp_text value "100Ω" (at 5.1 0.1) (layer "F.SilkS")
       (effects (font (size 1 1) (thickness 0.15)))
     )
@@
       (effects (font (size 0.75 0.75) (thickness 0.1)))
     )
-    (fp_text value "10Ω RC" (at 5.18 0) (layer "F.SilkS")
+    (fp_text value "10Ω" (at 5.18 0) (layer "F.SilkS")
       (effects (font (size 1 1) (thickness 0.15)))
     )
@@
       (effects (font (size 0.75 0.75) (thickness 0.1)))
     )
-    (fp_text value "100Ω_CharliePlex3" (at 5.1 0) (layer "F.SilkS")
+    (fp_text value "100Ω" (at 5.1 0) (layer "F.SilkS")
       (effects (font (size 1 1) (thickness 0.15)))
     )
@@
       (effects (font (size 0.75 0.75) (thickness 0.1)))
     )
-    (fp_text value "10kΩ PD pull-down" (at 5.1 -0.1) (layer "F.SilkS")
+    (fp_text value "10kΩ" (at 5.1 -0.1) (layer "F.SilkS")
       (effects (font (size 1 1) (thickness 0.15)))
     )
@@
       (effects (font (size 0.75 0.75) (thickness 0.1)))
     )
-    (fp_text value "1nF RC" (at 0.9726 2.9) (layer "F.SilkS")
+    (fp_text value "1nF" (at 0.9726 2.9) (layer "F.SilkS")
       (effects (font (size 1 1) (thickness 0.15)))
     )
@@
       (effects (font (size 0.75 0.75) (thickness 0.1)))
     )
-    (fp_text value "100Ω_CharliePlex2" (at 5.08 0) (layer "F.SilkS")
+    (fp_text value "100Ω" (at 5.08 0) (layer "F.SilkS")
       (effects (font (size 1 1) (thickness 0.15)))
     )
@@
       (effects (font (size 0.75 0.75) (thickness 0.1)))
     )
-    (fp_text value "100Ω Spike-LED" (at 5.08 0.1 180) (layer "F.SilkS")
+    (fp_text value "100Ω" (at 5.08 0.1 180) (layer "F.SilkS")
       (effects (font (size 1 1) (thickness 0.15)))
     )
@@
       (effects (font (size 0.75 0.75) (thickness 0.1)))
     )
-    (fp_text value "100Ω_CharliePlex1" (at 5 0.1) (layer "F.SilkS")
+    (fp_text value "100Ω" (at 5 0.1) (layer "F.SilkS")
       (effects (font (size 1 1) (thickness 0.15)))
     )
@@
       (effects (font (size 1.001047 1.001047) (thickness 0.15)))
     )
-    (fp_line (start -13.95 -27.15) (end 13.95 -27.15) (layer "F.SilkS") (width 0.127))
-    (fp_line (start 13.95 27.25) (end -13.95 27.25) (layer "F.SilkS") (width 0.127))
-    (fp_line (start 13.95 -27.15) (end 13.95 27.25) (layer "F.SilkS") (width 0.127))
     (fp_line (start -13.95 27.25) (end -13.95 -27.15) (layer "F.SilkS") (width 0.127))
+    (fp_line (start 13.95 -27.15) (end 13.95 27.25) (layer "F.SilkS") (width 0.127))
+    (fp_line (start 13.95 27.25) (end -13.95 27.25) (layer "F.SilkS") (width 0.127))
+    (fp_line (start -13.95 -27.15) (end 13.95 -27.15) (layer "F.SilkS") (width 0.127))
     (fp_line (start -14.2 27.5) (end -14.2 -27.4) (layer "F.CrtYd") (width 0.05))
-    (fp_line (start 14.2 -27.4) (end 14.2 27.5) (layer "F.CrtYd") (width 0.05))
-    (fp_line (start -14.2 -27.4) (end 14.2 -27.4) (layer "F.CrtYd") (width 0.05))
     (fp_line (start 14.2 27.5) (end -14.2 27.5) (layer "F.CrtYd") (width 0.05))
-    (fp_line (start 13.95 -27.15) (end 13.95 27.25) (layer "F.Fab") (width 0.127))
-    (fp_line (start 13.95 27.25) (end -13.95 27.25) (layer "F.Fab") (width 0.127))
+    (fp_line (start -14.2 -27.4) (end 14.2 -27.4) (layer "F.CrtYd") (width 0.05))
+    (fp_line (start 14.2 -27.4) (end 14.2 27.5) (layer "F.CrtYd") (width 0.05))
     (fp_line (start -13.95 27.25) (end -13.95 -27.15) (layer "F.Fab") (width 0.127))
+    (fp_line (start 13.95 27.25) (end -13.95 27.25) (layer "F.Fab") (width 0.127))
+    (fp_line (start 13.95 -27.15) (end 13.95 27.25) (layer "F.Fab") (width 0.127))
     (fp_line (start -13.95 -27.15) (end 13.95 -27.15) (layer "F.Fab") (width 0.127))
     (fp_circle (center -14.6 -19.9) (end -14.46 -19.9) (layer "F.Fab") (width 0.28) (fill none))
