File: V 2.2/PCB/Spikeling_V2.2.kicad_sch (KiCad schematic)
At the start: 44 parts, among them U1 ESP32-DEVKITC-32D, U2 MCP3208, U3 MCP3208

Commit message: update pcb
Parts:
- BZ1: renamed from Spike_Buzzer; value BZ1 -> (none); footprint Buzzer_Beeper:Buzzer_11.5x9.5RM5 -> (none)
- C1: value 1 μF -> (none); footprint Capacitor_THT:CP_Radial_D4.0mm_P2.00mm -> (none)
- C3: renamed from 1nF_RC1; value C3 -> (none); footprint Capacitor_THT:CP_Radial_D4.0mm_P2.00mm -> (none)
- D1: renamed from Photodiode1; value D1 -> (none); footprint LED_THT:LED_D5.0mm -> (none)
- D10: renamed from Mode9; value D10 -> (none); footprint LED_THT:LED_D3.0mm -> (none)
- D11: renamed from Mode10; value D11 -> (none); footprint LED_THT:LED_D3.0mm -> (none)
- D12: renamed from Mode11; value D12 -> (none); footprint LED_THT:LED_D3.0mm -> (none)
- D13: renamed from Mode12; value D13 -> (none); footprint LED_THT:LED_D3.0mm -> (none)
- D14: renamed from Spike_LED; value RGB -> (none); footprint LED_THT:LED_D5.0mm-4_RGB -> (none)
- D2: renamed from Mode1; value D2 -> (none); footprint LED_THT:LED_D3.0mm -> (none)
- D3: renamed from Mode2; value D3 -> (none); footprint LED_THT:LED_D3.0mm -> (none)
- D4: renamed from Mode3; value D4 -> (none); footprint LED_THT:LED_D3.0mm -> (none)
- D5: renamed from Mode4; value D5 -> (none); footprint LED_THT:LED_D3.0mm -> (none)
- D6: renamed from Mode5; value D6 -> (none); footprint LED_THT:LED_D3.0mm -> (none)
- D7: renamed from Mode6; value D7 -> (none); footprint LED_THT:LED_D3.0mm -> (none)
- D8: renamed from Mode7; value D8 -> (none); footprint LED_THT:LED_D3.0mm -> (none)
- D9: renamed from Mode8; value LED -> (none); footprint LED_THT:LED_D3.0mm -> (none)
- R1: renamed from 10Ω_RC1; value R1 -> (none); footprint Resistor_THT:R_Axial_DIN0207_L6.3mm_D2.5mm_P10.16mm_Horizontal -> (none)
- R2: renamed from 10kΩ_PD_pull-down1; value R2 -> (none); footprint Resistor_THT:R_Axial_DIN0207_L6.3mm_D2.5mm_P10.16mm_Horizontal -> (none)
- R3: renamed from 100Ω_Stim-LED1; value R3 -> (none); footprint Resistor_THT:R_Axial_DIN0207_L6.3mm_D2.5mm_P10.16mm_Horizontal -> (none)
- R4: renamed from 100Ω_Spike-LED1; value R4 -> (none); footprint Resistor_THT:R_Axial_DIN0207_L6.3mm_D2.5mm_P10.16mm_Horizontal -> (none)
- R5: renamed from 10kΩ_SW_pull-down1; value R5 -> (none); footprint Resistor_THT:R_Axial_DIN0207_L6.3mm_D2.5mm_P10.16mm_Horizontal -> (none)
- R6: renamed from 100Ω_CharliePlex1; value R6 -> (none); footprint Resistor_THT:R_Axial_DIN0207_L6.3mm_D2.5mm_P10.16mm_Horizontal -> (none)
- R7: renamed from 100Ω_CharliePlex2; value R7 -> (none); footprint Resistor_THT:R_Axial_DIN0207_L6.3mm_D2.5mm_P10.16mm_Horizontal -> (none)
- R8: renamed from 100Ω_CharliePlex3; value R8 -> (none); footprint Resistor_THT:R_Axial_DIN0207_L6.3mm_D2.5mm_P10.16mm_Horizontal -> (none)
- R9: renamed from 100Ω_CharliePlex4; value R9 -> (none); footprint Resistor_THT:R_Axial_DIN0207_L6.3mm_D2.5mm_P10.16mm_Horizontal -> (none)
- RV1: renamed from Synapse_1_Gain1; value RV1 -> (none); footprint Potentiometer_THT:Spikeling Potentiometer -> (none)
- RV2: renamed from Synapse_2_Gain1; value RV2 -> (none); footprint Potentiometer_THT:Spikeling Potentiometer -> (none)
- RV3: renamed from Voltage_Membrane1; value RV3 -> (none); footprint Potentiometer_THT:Spikeling Potentiometer -> (none)
- RV4: renamed from Noise1; value RV4 -> (none); footprint Potentiometer_THT:Spikeling Potentiometer -> (none)
- RV5: renamed from Photodiode_Gain1; value RV5 -> (none); footprint Potentiometer_THT:Spikeling Potentiometer -> (none)
- RV6: renamed from Stimulus_Strength1; value RV6 -> (none); footprint Potentiometer_THT:Spikeling Potentiometer -> (none)
- RV7: renamed from Stimulus_Frequency1; value RV7 -> (none); footprint Potentiometer_THT:Spikeling Potentiometer -> (none)
- SW1: renamed from Mode_Button1; value SW1 -> (none); footprint Button_Switch_THT:SW_PUSH_6mm_H13mm -> (none)
- SW2: renamed from Reset_Button1; value SW2 -> (none); footprint Button_Switch_THT:Spikeling reset button -> (none)
- renumbered Synapse_Out to J1, Synapse_In_1 to J2, Synapse_in_2 to J3, Current_In1 to J4, StimulusOut to J5
